Commit message: Add files via upload

File: aruco_sim_rover/urdf/aruco_marker.xacro (robot description, xacro)
@@ -3,5 +3,5 @@
 	<xacro:property name="robot_name" value="aruco_marker" />
 	<xacro:property name="pole_mass" value="0"/>
-	<xacro:property name="pole_height" value="1"/>
+	<xacro:property name="pole_height" value="0.6"/>
 	<xacro:property name="pole_radius" value=".015"/>
 	<xacro:property name="marker_mass" value=".240"/>
@@ -46,5 +46,5 @@
 			<origin xyz="0 0 0" rpy="0 0 0"/>
 			<geometry>
-				<mesh filename="package://aruco_sim/meshes/$(arg model_file)"/>
+				<mesh filename="package://aruco_sim_rover/meshes/$(arg model_file)"/>
 			</geometry>
 		</visual>
