Commit message: TF Fix

File: rover_description/urdf/rover_description.urdf (robot description, URDF)
Before this commit: robot mars_rover, 11 links, 10 joints
Links:
- added link base_footprint
- added link chassis, mass 14.4435926271869; collision mesh filename=package://rover_description/meshes/base_link.STL; visual mesh filename=package://rover_description/meshes/base_link.STL
- link base_link: mass 14.4435926271869 -> None; geometry 
Joints:
- added joint base_footprint_tf: type fixed, parent base_link, child base_footprint, origin xyz=0 0 0 rpy=0 0 0
- added joint connector: type fixed, parent base_link, child chassis, origin xyz=0 0 0.4 rpy=0 0 0
- joint camera_joint: parent base_link -> chassis
- joint imu_joint: parent base_link -> chassis
- joint steer1: parent base_link -> chassis
- joint steer2: parent base_link -> chassis
- joint steer4: parent base_link -> chassis
- joint steer_3: parent base_link -> chassis

Commit message: worlds updates and optical link

File: rover_description/urdf/rover_description.urdf (robot description, URDF)
Before this commit: robot mars_rover, 13 links, 12 joints
Links:
- added link camera_optical_link
Joints:
- added joint camera_optical_joint: type fixed, parent camera_link, child camera_optical_link, origin xyz=0.1 0 0.1 rpy=-1.57 0 -1.57

Commit message: Updated

File: rover_description/urdf/rover_description.urdf (robot description, URDF)
Before this commit: robot mars_rover, 14 links, 13 joints
Links:
- added link camera_link_1; collision box size=0.1 0.1 0.1; visual box size=0.1 0.1 0.1
- added link camera_link_2; collision box size=0.1 0.1 0.1; visual box size=0.1 0.1 0.1
- added link camera_optical_link_1
- added link camera_optical_link_2
- link wheel1: geometry collision cylinder length=0.144 radius=0.11; visual mesh filename=package://rover_description/meshes/wheel1.STL
- link wheel2: geometry collision cylinder length=0.144 radius=0.11; visual mesh filename=package://rover_description/meshes/wheel2.STL
- link wheel3: geometry collision cylinder length=0.144 radius=0.11; visual mesh filename=package://rover_description/meshes/wheel3.STL
- link wheel4: geometry collision cylinder length=0.144 radius=0.11; visual mesh filename=package://rover_description/meshes/wheel4.STL
Joints:
- added joint camera_joint_1: type fixed, parent chassis, child camera_link_1, origin xyz=0 0.24 0.1 rpy=0 0 1.57
- added joint camera_joint_2: type fixed, parent chassis, child camera_link_2, origin xyz=0 -0.24 0.1 rpy=0 0 -1.57
- added joint camera_optical_joint_1: type fixed, parent camera_link_1, child camera_optical_link_1, origin xyz=0 0 0 rpy=-1.57 0 -1.57
- added joint camera_optical_joint_2: type fixed, parent camera_link_2, child camera_optical_link_2, origin xyz=0 0 0 rpy=-1.57 0 -1.57
- joint camera_optical_joint: origin xyz=0.1 0 0.1 rpy=-1.57 0 -1.57 -> xyz=0 0 0 rpy=-1.57 0 -1.57
- joint steer1: limit lower=-1.57 upper=1.57 effort=5 velocity=6.28 -> lower=-1.57 upper=1.57 effort=10 velocity=6.28
- joint steer2: limit lower=-1.57 upper=1.57 effort=5 velocity=6.28 -> lower=-1.57 upper=1.57 effort=10 velocity=6.28
- joint steer4: limit lower=-1.57 upper=1.57 effort=5 velocity=6.28 -> lower=-1.57 upper=1.57 effort=10 velocity=6.28
- joint steer_3: limit lower=-1.57 upper=1.57 effort=5 velocity=6.28 -> lower=-1.57 upper=1.57 effort=10 velocity=6.28

Commit message: my part

File: rover_description/urdf/rover_description.urdf (robot description, URDF)
Before this commit: robot mars_rover, 18 links, 17 joints
Links:
- link camera_link: mass None -> 0.01; geometry collision box size=0.05 0.05 0.05; visual box size=0.05 0.05 0.05
- link camera_link_1: mass None -> 0.01; geometry collision box size=0.05 0.05 0.05; visual box size=0.05 0.05 0.05
- link camera_link_2: mass None -> 0.01; geometry collision box size=0.05 0.05 0.05; visual box size=0.05 0.05 0.05
- link imu_link: mass None -> 0.001; geometry visual box size=0.02 0.02 0.01
Joints:
- joint imu_joint: origin (none) -> xyz=0.0 0.0 0.0 rpy=0 0 0
